Commit message: only reorder in and out the network

File: src/robots/g1_description/urdf/g1_29dof_rev_1_0_modify_inertia.urdf (robot description, URDF)
Before this commit: robot g1_29dof_rev_1_0, 40 links, 39 joints
Links:
- link left_knee_link: geometry visual mesh filename=package://g1_description/meshes/left_knee_link.STL
- link right_knee_link: geometry visual mesh filename=package://g1_description/meshes/right_knee_link.STL
